File: src/H0001-Solenoid-Driver/H0001-Solenoid-Driver.kicad_pcb (KiCad board)
At the start: 2 copper layers, 75.2 x 35.4 mm, 19 parts, among them K1 AQH0223AX, K2 AQH0223AX, P1 647676-2, P2 647676-3, P3 647676-3, P4 647676-3

Commit message: minor local commits
Routing:
- net Net-(C2-Pad1): track 21.9 -> 37.4 mm
Changed lines of the file:
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@@
     (pad_to_mask_clearance 0)
     (pcbplotparams
-      (layerselection 0x00010fc_ffffffff)
+      (layerselection 0x003d0fc_ffffffff)
       (disableapertmacros false)
       (usegerberextensions false)
@@
       (outputformat 1)
       (mirror false)
-      (drillshape 1)
+      (drillshape 0)
       (scaleselection 1)
-      (outputdirectory "")
+      (outputdirectory "../../production/")
     )
   )
@@
   (segment (start 116.84 78.3425) (end 120.7427 78.3425) (width 0.254) (layer "F.Cu") (net 1))
   (segment (start 106.3752 76.043799) (end 110.841799 76.043799) (width 0.254) (layer "F.Cu") (net 2))
-  (segment (start 103.3272 92.3544) (end 103.3272 88.6968) (width 0.254) (layer "F.Cu") (net 3))
+  (segment (start 110.2868 91.9988) (end 116.332 98.044) (width 0.254) (layer "F.Cu") (net 3))
   (segment (start 116.586 97.9005) (end 125.5357 97.9005) (width 0.254) (layer "F.Cu") (net 3))
+  (segment (start 103.3272 92.3544) (end 103.3272 91.9988) (width 0.254) (layer "F.Cu") (net 3))
   (segment (start 103.3272 88.6968) (end 104.8512 87.1728) (width 0.254) (layer "F.Cu") (net 3))
   (segment (start 104.8512 87.1728) (end 105.3084 87.1728) (width 0.254) (layer "F.Cu") (net 3))
   (segment (start 100.2816 95.4) (end 103.3272 92.3544) (width 0.254) (layer "F.Cu") (net 3))
+  (segment (start 105.1052 91.9988) (end 110.2868 91.9988) (width 0.254) (layer "F.Cu") (net 3))
   (segment (start 97.915 95.4) (end 100.2816 95.4) (width 0.254) (layer "F.Cu") (net 3))
+  (segment (start 103.3272 91.9988) (end 103.3272 88.6968) (width 0.254) (layer "F.Cu") (net 3))
+  (segment (start 103.3272 91.9988) (end 105.1052 91.9988) (width 0.254) (layer "F.Cu") (net 3))
   (segment (start 107.387399 90.173801) (end 108.3564 89.2048) (width 0.254) (layer "F.Cu") (net 4))
   (segment (start 108.3564 89.2048) (end 110.0328 89.2048) (width 0.254) (layer "F.Cu") (net 4))
